File: Gyro.sch (KiCad schematic (older format))
At the start: 4 parts, among them U7 MPU-6000

Commit message: Moved GND symbol slightly
Other:
- moved on the sheet: C46
Changed lines of the file:
@@
 L Device:C_Small C?
 U 1 1 60B2E47E
-P 6350 4000
+P 6450 4000
 AR Path="/60B2E47E" Ref="C?"  Part="1"
 AR Path="/60B2ABA4/60B2E47E" Ref="C46"  Part="1"
-F 0 "C46" V 6400 3850 50  0000 L CNN
-F 1 "2.2uF" V 6250 3850 50  0000 L CNN
-F 2 "Capacitor_SMD:C_0402_1005Metric" H 6350 4000 50  0001 C CNN
-F 3 "~" H 6350 4000 50  0001 C CNN
-	1    6350 4000
+F 0 "C46" V 6500 3850 50  0000 L CNN
+F 1 "2.2uF" V 6350 3850 50  0000 L CNN
+F 2 "Capacitor_SMD:C_0402_1005Metric" H 6450 4000 50  0001 C CNN
+F 3 "~" H 6450 4000 50  0001 C CNN
+	1    6450 4000
 	0    -1   -1   0
 $EndComp
@@
 L power:GND #PWR?
 U 1 1 60B2E484
-P 6450 4000
+P 6650 4150
 AR Path="/60B2E484" Ref="#PWR?"  Part="1"
 AR Path="/60B2ABA4/60B2E484" Ref="#PWR0167"  Part="1"
-F 0 "#PWR0167" H 6450 3750 50  0001 C CNN
-F 1 "GND" V 6455 3872 50  0000 R CNN
-F 2 "" H 6450 4000 50  0001 C CNN
-F 3 "" H 6450 4000 50  0001 C CNN
-	1    6450 4000
-	0    -1   -1   0
+F 0 "#PWR0167" H 6650 3900 50  0001 C CNN
+F 1 "GND" H 6800 4000 50  0000 R CNN
+F 2 "" H 6650 4150 50  0001 C CNN
+F 3 "" H 6650 4150 50  0001 C CNN
+	1    6650 4150
+	1    0    0    -1
 $EndComp
-Wire Wire Line
-	6250 4000 6200 4000
 $Comp
 L power:GND #PWR?
@@
 Text HLabel 4800 3800 0    50   Input ~ 0
 SPI1_CS
+Wire Wire Line
+	6650 4000 6650 4150
+Wire Wire Line
+	6200 4000 6350 4000
+Wire Wire Line
+	6550 4000 6650 4000
 $EndSCHEMATC
